Commit message: fit to gazebo

File: models/gazebo_blackship.xacro (robot description, xacro)
@@ -31,5 +31,5 @@
             <inertial>
                 <origin xyz="0 0 0" rpy="0 0 0"/>
-                <mass value="10"/>
+                <mass value="20"/>
                 <inertia ixx="1.0" ixy="0.0" ixz="0.0"
                          iyy="1.0" iyz="0.0"
