Commit message: update for inertia

File: models/blackship.xacro (robot description, xacro)
@@ -23,4 +23,15 @@
                 </material>
             </visual>
+            <collision>
+                <origin xyz="0 0 0" rpy="0 0 0"/>
+                <geometry>
+                    <box size="${blackship_body_depth} ${blackship_body_width} ${blackship_body_height}"/>
+                </geometry>
+            </collision>
+            <inertial>
+                <origin xyz="0 0 0" rpy="0 0 0"/>
+                <mass value="${blackship_body_weight}"/>
+                <xacro:insert_block name="blackship_body_inertia"/>
+            </inertial>
         </link>
         <xacro:blackship_wheels

File: models/blackship_wheels.xacro (robot description, xacro)
@@ -22,4 +22,16 @@
                 </material>
             </visual>
+            <collision>
+                <origin rpy="${DEG2RAD*90} 0 0" xyz="0 0 0"/>
+                <geometry>
+                    <cylinder radius="${blackship_wheel_radius}"
+                              length="${blackship_wheel_width}"/>
+                </geometry>
+            </collision>
+            <inertial>
+                <origin rpy="${DEG2RAD*90} 0 0" xyz="0 0 0"/>
+                <mass value="${blackship_wheel_weight}"/>
+                <xacro:insert_block name="blackship_wheel_inertia"/>
+            </inertial>
         </link>
         <joint name="${joint_blackship_wheel}_${suffix}_2" type="fixed">

File: models/property.xacro (robot description, xacro)
@@ -2,5 +2,5 @@
 <robot>
     <!--SEE http://homepage3.nifty.com/orangejuice/-->
-    <!--All values are in [m]-->
+    <!--All values are in [m][kg]-->
     <!--x is radius-->
     <property name="blackship_body_depth" value="0.600"/>
@@ -17,3 +17,20 @@
     <property name="blackship_topboard_width" value="${blackship_body_width}"/>
     <property name="blackship_topboard_height" value="0.003"/>
+    <!--==========================================================-->
+    <property name="blackship_body_weight" value="20"/>
+    <property name="blackship_body_inertia">
+        <inertia
+                ixx="${(1.0/3.0)*blackship_body_weight*(blackship_body_width*blackship_body_width + blackship_body_height*blackship_body_height)}"
+                iyy="${(1.0/3.0)*blackship_body_weight*(blackship_body_height*blackship_body_height + blackship_body_depth*blackship_body_depth)}"
+                izz="${(1.0/3.0)*blackship_body_weight*(blackship_body_depth*blackship_body_depth + blackship_body_width*blackship_body_width)}"
+                ixy="0.0" ixz="0.0" iyz="0.0"/>
+    </property>
+    <property name="blackship_wheel_weight" value="0.8"/>
+    <property name="blackship_wheel_inertia">
+        <inertia
+                ixx="${(1.0/4.0)*blackship_wheel_weight*(blackship_wheel_radius*blackship_wheel_radius + (1.0/3.0)*blackship_wheel_width*blackship_wheel_width)}"
+                iyy="${(1.0/4.0)*blackship_wheel_weight*(blackship_wheel_radius*blackship_wheel_radius + (1.0/3.0)*blackship_wheel_width*blackship_wheel_width)}"
+                izz="${(1.0/2.0)*blackship_wheel_weight*(blackship_wheel_radius*blackship_wheel_radius)}"
+                ixy="0.0" ixz="0.0" iyz="0.0"/>
+    </property>
 </robot>

Commit message: prepare for gazebo_plugin

File: models/blackship.xacro (robot description, xacro)
@@ -30,5 +30,5 @@
             </collision>
             <inertial>
-                <origin xyz="0 0 0" rpy="0 0 0"/>
+                <origin xyz="0 0 ${-blackship_body_height/2}" rpy="0 0 0"/>
                 <mass value="${blackship_body_weight}"/>
                 <xacro:insert_block name="blackship_body_inertia"/>

File: models/blackship_wheels.xacro (robot description, xacro)
@@ -6,10 +6,11 @@
     <xacro:macro name="blackship_wheel"
                  params="parent_link suffix *origin">
-        <joint name="${joint_blackship_wheel}_${suffix}" type="fixed">
+        <joint name="${joint_blackship_wheel}_${suffix}" type="continuous">
+            <axis xyz="0 1 0"/>
             <insert_block name="origin"/>
             <parent link="${parent_link}"/>
-            <child link="${link_blackship_wheel}_${suffix}"/>
+            <child link="${link_blackship_wheel}_1_${suffix}"/>
         </joint>
-        <link name="${link_blackship_wheel}_${suffix}">
+        <link name="${link_blackship_wheel}_1_${suffix}">
             <visual>
                 <origin rpy="${DEG2RAD*90} 0 0" xyz="0 0 0"/>
@@ -35,10 +36,10 @@
             </inertial>
         </link>
-        <joint name="${joint_blackship_wheel}_${suffix}_2" type="fixed">
+        <joint name="${joint_blackship_wheel}_2_${suffix}" type="fixed">
             <origin rpy="0 0 0" xyz="0 0 0"/>
-            <parent link="${link_blackship_wheel}_${suffix}"/>
-            <child link="${link_blackship_wheel}_${suffix}_2"/>
+            <parent link="${link_blackship_wheel}_1_${suffix}"/>
+            <child link="${link_blackship_wheel}_2_${suffix}"/>
         </joint>
-        <link name="${link_blackship_wheel}_${suffix}_2">
+        <link name="${link_blackship_wheel}_2_${suffix}">
             <visual>
                 <origin rpy="${DEG2RAD*90} 0 0" xyz="0 0 0"/>

File: models/config.xacro (robot description, xacro)
@@ -11,3 +11,26 @@
     <property name="link_blackship_topboard" value="link_blackship_topboard"/>
     <property name="link_blackship_offset_center" value="link_blackship_offset_center"/>
+    <property name="link_mico_base" value="mico_link_base"/>
+    <property name="link_mico_1" value="mico_link_1"/>
+    <property name="link_mico_2" value="mico_link_2"/>
+    <property name="link_mico_3" value="mico_link_3"/>
+    <property name="link_mico_4" value="mico_link_4"/>
+    <property name="link_mico_5" value="mico_link_5"/>
+    <property name="link_mico_hand" value="mico_link_hand"/>
+    <property name="link_mico_finger_1" value="finger_proximal_limb_1"/>
+    <property name="link_mico_finger_2" value="finger_proximal_limb_2"/>
+    <property name="link_mico_finger_tip_1" value="finger_distal_limb_1"/>
+    <property name="link_mico_finger_tip_2" value="finger_distal_limb_2"/>
+    <property name="mico_api_origin" value="mico_api_origin"/>
+    <property name="joint_mico_base" value="mico_joint_base"/>
+    <property name="joint_mico_1" value="mico_joint_1"/>
+    <property name="joint_mico_2" value="mico_joint_2"/>
+    <property name="joint_mico_3" value="mico_joint_3"/>
+    <property name="joint_mico_4" value="mico_joint_4"/>
+    <property name="joint_mico_5" value="mico_joint_5"/>
+    <property name="joint_mico_6" value="mico_joint_6"/>
+    <property name="joint_mico_finger_1" value="mico_joint_finger_1"/>
+    <property name="joint_mico_finger_tip_1" value="mico_joint_finger_tip_1"/>
+    <property name="joint_mico_finger_2" value="mico_joint_finger_2"/>
+    <property name="joint_mico_finger_tip_2" value="mico_joint_finger_tip_2"/>
 </robot>
