Commit message: prepare for changing file tree

File: models/blackship_wheels.xacro (robot description, xacro)
@@ -7,8 +7,9 @@
                  params="parent_link suffix *origin">
         <joint name="${joint_blackship_wheel}_${suffix}" type="continuous">
-            <axis xyz="0 1 0"/>
+            <axis xyz="0 1 0" rpy="0 0 0"/>
             <insert_block name="origin"/>
             <parent link="${parent_link}"/>
             <child link="${link_blackship_wheel}_1_${suffix}"/>
+            <joint_properties damping="0.0" friction="0.0"/>
         </joint>
         <link name="${link_blackship_wheel}_1_${suffix}">

File: models/property.xacro (robot description, xacro)
@@ -26,10 +26,10 @@
                 ixy="0.0" ixz="0.0" iyz="0.0"/>
     </property>
-    <property name="blackship_wheel_weight" value="0.8"/>
+    <property name="blackship_wheel_weight" value="3"/>
     <property name="blackship_wheel_inertia">
         <inertia
                 ixx="${(1.0/4.0)*blackship_wheel_weight*(blackship_wheel_radius*blackship_wheel_radius + (1.0/3.0)*blackship_wheel_width*blackship_wheel_width)}"
-                iyy="${(1.0/4.0)*blackship_wheel_weight*(blackship_wheel_radius*blackship_wheel_radius + (1.0/3.0)*blackship_wheel_width*blackship_wheel_width)}"
-                izz="${(1.0/2.0)*blackship_wheel_weight*(blackship_wheel_radius*blackship_wheel_radius)}"
+                iyy="${(1.0/2.0)*blackship_wheel_weight*(blackship_wheel_radius*blackship_wheel_radius)}"
+                izz="${(1.0/4.0)*blackship_wheel_weight*(blackship_wheel_radius*blackship_wheel_radius + (1.0/3.0)*blackship_wheel_width*blackship_wheel_width)}"
                 ixy="0.0" ixz="0.0" iyz="0.0"/>
     </property>
