Commit message: make sure it works under gazebo2

File: bs_model/models/blackship.urdf.xacro (robot description, xacro)
@@ -1,5 +1,8 @@
 <?xml version="1.0"?>
 <robot name="blackship" xmlns:xacro="http://www.ros.org/wiki/xacro">
-    <xacro:include filename="$(find ros_blackship)/models/blackship.xacro"/>
+    <xacro:include filename="$(find bs_model)/models/blackship.xacro"/>
+    <xacro:if value="$(arg is_gazebo)">
+        <xacro:include filename="$(find bs_simulator)/gazebo/blackship.gazebo"/>
+    </xacro:if>
     <link name="blackship_root"/>
     <xacro:blackship parent_link="blackship_root"/>

File: bs_model/models/blackship.xacro (robot description, xacro)
@@ -1,9 +1,9 @@
 <?xml version="1.0"?>
 <robot xmlns:xacro="http://www.ros.org/wiki/xacro">
-    <xacro:include filename="$(find ros_blackship)/models/define.xacro"/>
-    <xacro:include filename="$(find ros_blackship)/models/config.xacro"/>
-    <xacro:include filename="$(find ros_blackship)/models/property.xacro"/>
-    <xacro:include filename="$(find ros_blackship)/models/blackship_wheels.xacro"/>
-    <xacro:include filename="$(find ros_blackship)/models/blackship_topboard.xacro"/>
+    <xacro:include filename="$(find bs_model)/models/define.xacro"/>
+    <xacro:include filename="$(find bs_model)/models/config.xacro"/>
+    <xacro:include filename="$(find bs_model)/models/property.xacro"/>
+    <xacro:include filename="$(find bs_model)/models/blackship_wheels.xacro"/>
+    <xacro:include filename="$(find bs_model)/models/blackship_topboard.xacro"/>
     <xacro:macro name="blackship" params="parent_link">
         <joint name="${joint_blackship_body}" type="fixed">

File: bs_model/models/blackship_topboard.xacro (robot description, xacro)
@@ -1,7 +1,7 @@
 <?xml version="1.0"?>
 <robot xmlns:xacro="http://www.ros.org/wiki/xacro">
-    <xacro:include filename="$(find ros_blackship)/models/define.xacro"/>
-    <xacro:include filename="$(find ros_blackship)/models/config.xacro"/>
-    <xacro:include filename="$(find ros_blackship)/models/property.xacro"/>
+    <xacro:include filename="$(find bs_model)/models/define.xacro"/>
+    <xacro:include filename="$(find bs_model)/models/config.xacro"/>
+    <xacro:include filename="$(find bs_model)/models/property.xacro"/>
     <xacro:macro name="blackship_offset_pole"
                  params="parent_link suffix *origin">

File: bs_model/models/blackship_wheels.xacro (robot description, xacro)
@@ -1,7 +1,7 @@
 <?xml version="1.0"?>
 <robot xmlns:xacro="http://www.ros.org/wiki/xacro">
-    <xacro:include filename="$(find ros_blackship)/models/define.xacro"/>
-    <xacro:include filename="$(find ros_blackship)/models/config.xacro"/>
-    <xacro:include filename="$(find ros_blackship)/models/property.xacro"/>
+    <xacro:include filename="$(find bs_model)/models/define.xacro"/>
+    <xacro:include filename="$(find bs_model)/models/config.xacro"/>
+    <xacro:include filename="$(find bs_model)/models/property.xacro"/>
     <xacro:macro name="blackship_wheel"
                  params="parent_link suffix *origin">
@@ -12,4 +12,5 @@
             <child link="${link_blackship_wheel}_1_${suffix}"/>
             <joint_properties damping="0.0" friction="0.0"/>
+            <limit effort="100" velocity="100"/>
         </joint>
         <link name="${link_blackship_wheel}_1_${suffix}">
@@ -37,5 +38,6 @@
             </inertial>
         </link>
-        <joint name="${joint_blackship_wheel}_2_${suffix}" type="fixed">
+        <joint name="${joint_blackship_wheel}_2_${suffix}" type="continuous">
+            <axis xyz="0 1 0" rpy="0 0 0"/>
             <origin rpy="0 0 0" xyz="0 0 0"/>
             <parent link="${link_blackship_wheel}_1_${suffix}"/>

File: bs_model/models/property.xacro (robot description, xacro)
@@ -26,5 +26,5 @@
                 ixy="0.0" ixz="0.0" iyz="0.0"/>
     </property>
-    <property name="blackship_wheel_weight" value="3"/>
+    <property name="blackship_wheel_weight" value="1"/>
     <property name="blackship_wheel_inertia">
         <inertia
