Commit message: enable to visualize sporks of bs

File: bs_model/models/blackship_wheels.xacro (robot description, xacro)
@@ -38,5 +38,5 @@
             </inertial>
         </link>
-        <joint name="${joint_blackship_wheel}_2_${suffix}" type="continuous">
+        <joint name="${joint_blackship_wheel}_2_${suffix}" type="fixed">
             <axis xyz="0 1 0" rpy="0 0 0"/>
             <origin rpy="0 0 0" xyz="0 0 0"/>

Commit message: add inputVelTopicName tag

File: bs_model/models/blackship_wheels.xacro (robot description, xacro)
@@ -4,7 +4,11 @@
     <xacro:include filename="$(find bs_model)/models/config.xacro"/>
     <xacro:include filename="$(find bs_model)/models/property.xacro"/>
+    <property name="wheel_type" value="continuous"/>
+    <!--<xacro:unless value="$(arg is_gazebo)">-->
+        <!--<property name="wheel_type" value="fixed"/>-->
+    <!--</xacro:unless>-->
     <xacro:macro name="blackship_wheel"
                  params="parent_link suffix *origin">
-        <joint name="${joint_blackship_wheel}_${suffix}" type="continuous">
+        <joint name="${joint_blackship_wheel}_${suffix}" type="${wheel_type}">
             <axis xyz="0 1 0" rpy="0 0 0"/>
             <insert_block name="origin"/>
